File: alicia-cook.kicad_pcb (KiCad board)
At the start: 2 copper layers, 291.8 x 91.8 mm, 109 parts, among them J1 02x05, J2 02x05, SW1 switch, SW10 switch, SW11 switch, SW12 switch, SW13 switch, SW14 switch, SW15 switch, SW16 switch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

Commit message: some wilding tracks smh my head.
Routing:
- net ROW2A: track 327.2 -> 328.9 mm
- net ROW3A: track 354.6 -> 356.2 mm

Commit message: some route fixes.
Parts:
- added H10: MountingHole, footprints:hole-three, F.Cu at (128.5, 50.8)
- added H11: MountingHole, footprints:hole-three, F.Cu at (137.0, 77.0)
- added H12: MountingHole, footprints:hole-three, F.Cu at (133.0, 77.0)
- added H9: MountingHole, footprints:hole-three, F.Cu at (124.5, 51.0)
- moved H2 2.41 mm to (128.4, 64.0)
- moved H5 2.26 mm to (124.5, 64.0)
- moved H3 1.00 mm to (128.4, 33.0)
Connections:
- J2 pad 5: ROW2A -> ROW2
- J2 pad 7: ROW3A -> ROW3
- U1 pad 19: ROW3A -> ROW3
- U1 pad 20: ROW2A -> ROW2
- diode15 pad 1: ROW2A -> ROW2
- diode16 pad 1: ROW2A -> ROW2
- diode17 pad 1: ROW2A -> ROW2
- diode18 pad 1: ROW2A -> ROW2
- diode19 pad 1: ROW2A -> ROW2
- diode20 pad 1: ROW2A -> ROW2
- diode21 pad 1: ROW2A -> ROW2
- diode22 pad 1: ROW3A -> ROW3
- diode24 pad 1: ROW3A -> ROW3
- diode25 pad 1: ROW3A -> ROW3
- diode26 pad 1: ROW3A -> ROW3
- diode27 pad 1: ROW3A -> ROW3
Routing:
- net ROW3: track 116.6 -> 773.8 mm
- net ROW2: track 122.3 -> 617.8 mm
- net ROW3A: track 356.2 -> 0.00 mm
- net ROW2A: track 328.9 -> 0.00 mm
Other:
- outline, holes or cut-outs redrawn
