File: alicia-cook.kicad_pcb (KiCad board)
At the start: 2 copper layers, 291.8 x 91.8 mm, 113 parts, among them J1 02x05, J2 02x05, SW1 switch, SW10 switch, SW11 switch, SW12 switch, SW13 switch, SW14 switch, SW15 switch, SW16 switch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

Commit message: 3d models.
Parts:
- D1, D10, D11, D12, D13, D14, D15, D16, D17, D18, D19, D2, D20, D21, D22, D23, D3, D4, D5, D6, D7, D8, D9, diode1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: footprint footprints:diode-vertical -> footprints:diode
- switch25: footprint footprints:15u-minimal -> footprints:1u-minimal
